File: Atari2600_Clone/Atari2600_Clone/Atari2600_Clone.sch (KiCad schematic (older format))
At the start: 8 parts, among them J1 Atari cartridge

Commit message: Two DB9s were added + A3 page format
Parts:
- added J1, J2: DB9_Male, symbol Connector:DB9_Male
- gave numbers to parts that had none: 3
Connections:
- net GND: now also U4.8 (VSS)
Other:
- moved on the sheet: D10, D9, J1, R1, R16, U1, U2, U4
